Commit message: tried addind cad file + triangles detection. coordinates of triangles are not stable, cant move propperly yet

File: urdf/ur5e_cube.urdf.xacro (robot description, xacro)
@@ -64,14 +64,16 @@
     <link name="cube">
     <visual>
-        <geometry>
-        <box size="0.5 0.5 0.5"/>
-        </geometry>
-        <material name="red">
-        <color rgba="1 0 0 1"/>
-        </material>
+      <geometry>
+        <mesh filename="file:///home/iku/ur5e_ws/src/ur5e_surface_path/meshes/tinkercadCube.stl"
+              scale="0.001 0.001 0.001"/>
+      </geometry>
+      <material name="red">
+      <color rgba="1 0 0 1"/>
+      </material>
     </visual>
     <collision>
         <geometry>
-        <box size="0.5 0.5 0.5"/>
+        <mesh filename="file:///home/iku/ur5e_ws/src/ur5e_surface_path/meshes/tinkercadCube.stl"
+              scale="0.001 0.001 0.001"/>
         </geometry>
     </collision>
@@ -84,5 +86,5 @@
     <parent link="world"/>
     <child link="cube"/>
-    <origin xyz="0.0 0.9 0.26" rpy="0 0 0"/>
+    <origin xyz="0.0 0.75 0.25" rpy="0 0 0"/>
     </joint>
   <gazebo reference="world">

Commit message: 50cm cube and claude getPose() variant. dont forget to use sim time

File: urdf/ur5e_cube.urdf.xacro (robot description, xacro)
@@ -65,5 +65,5 @@
     <visual>
       <geometry>
-        <mesh filename="file:///home/iku/ur5e_ws/src/ur5e_surface_path/meshes/tinkercadCube.stl"
+        <mesh filename="file:///home/iku/ur5e_ws/src/ur5e_surface_path/meshes/50cmCube.stl"
               scale="0.001 0.001 0.001"/>
       </geometry>
@@ -74,5 +74,5 @@
     <collision>
         <geometry>
-        <mesh filename="file:///home/iku/ur5e_ws/src/ur5e_surface_path/meshes/tinkercadCube.stl"
+        <mesh filename="file:///home/iku/ur5e_ws/src/ur5e_surface_path/meshes/50cmCube.stl"
               scale="0.001 0.001 0.001"/>
         </geometry>
@@ -86,5 +86,5 @@
     <parent link="world"/>
     <child link="cube"/>
-    <origin xyz="0.0 0.75 0.25" rpy="0 0 0"/>
+    <origin xyz="0.0 1.0 0.0" rpy="0 0 0"/>
     </joint>
   <gazebo reference="world">

Commit message: generalized file path; removed some folders

File: urdf/ur5e_cube.urdf.xacro (robot description, xacro)
@@ -65,5 +65,5 @@
     <visual>
       <geometry>
-        <mesh filename="file:///home/iku/ur5e_ws/src/ur5e_surface_path/meshes/50cmCube.stl"
+        <mesh filename="package://ur5e_surface_path/meshes/50cmCube.stl"
               scale="0.001 0.001 0.001"/>
       </geometry>
@@ -74,5 +74,5 @@
     <collision>
         <geometry>
-        <mesh filename="file:///home/iku/ur5e_ws/src/ur5e_surface_path/meshes/50cmCube.stl"
+        <mesh filename="package://ur5e_surface_path/meshes/50cmCube.stl"
               scale="0.001 0.001 0.001"/>
         </geometry>

Commit message: fixed: cube import

File: urdf/ur5e_cube.urdf.xacro (robot description, xacro)
@@ -65,5 +65,5 @@
     <visual>
       <geometry>
-        <mesh filename="package://ur5e_surface_path/meshes/50cmCube.stl"
+        <mesh filename="file://$(find ur5e_surface_path)/meshes/50cmCube.stl"
               scale="0.001 0.001 0.001"/>
       </geometry>
@@ -74,5 +74,5 @@
     <collision>
         <geometry>
-        <mesh filename="package://ur5e_surface_path/meshes/50cmCube.stl"
+        <mesh filename="file://$(find ur5e_surface_path)/meshes/50cmCube.stl"
               scale="0.001 0.001 0.001"/>
         </geometry>

Commit message: tinkercad model

File: urdf/ur5e_cube.urdf.xacro (robot description, xacro)
@@ -86,5 +86,5 @@
     <parent link="world"/>
     <child link="cube"/>
-    <origin xyz="0.0 1.0 0.0" rpy="0 0 0"/>
+    <origin xyz="0.0 0.65 0.0" rpy="0 0 0"/>
     </joint>
   <gazebo reference="world">

Commit message: tracing of a hemosphere

File: urdf/ur5e_cube.urdf.xacro (robot description, xacro)
@@ -86,5 +86,5 @@
     <parent link="world"/>
     <child link="cube"/>
-    <origin xyz="0.0 0.65 0.0" rpy="0 0 0"/>
+    <origin xyz="0.0 0.65 0.0" rpy="0 0 3.1415"/>
     </joint>
   <gazebo reference="world">
