Commit message: need to debug the run after the planning bc it does a wrong trajectory and add a for loop after it to show the coverage

File: urdf/ur5e_cube.urdf.xacro (robot description, xacro)
@@ -74,5 +74,5 @@
     <collision>
         <geometry>
-        <mesh filename="file://$(find ur5e_surface_path)/meshes/50cmCube.stl"
+        <mesh filename="file://$(find ur5e_surface_path)/meshes/50cmCubegg.stl"
               scale="0.001 0.001 0.001"/>
         </geometry>

Commit message: forgor to add?

File: urdf/ur5e_cube.urdf.xacro (robot description, xacro)
@@ -74,5 +74,5 @@
     <collision>
         <geometry>
-        <mesh filename="file://$(find ur5e_surface_path)/meshes/50cmCubegg.stl"
+        <mesh filename="file://$(find ur5e_surface_path)/meshes/50cmCube.stl"
               scale="0.001 0.001 0.001"/>
         </geometry>

Commit message: upto date with latest meeting before september

File: urdf/ur5e_cube.urdf.xacro (robot description, xacro)
@@ -86,5 +86,5 @@
     <parent link="world"/>
     <child link="cube"/>
-    <origin xyz="0.0 0.65 0.0" rpy="0 0 3.1415"/>
+    <origin xyz="0.0 0.65 0.2" rpy="0 0 3.1415"/>
     </joint>
   <gazebo reference="world">

Commit message: repeats some waypoints still

File: urdf/ur5e_cube.urdf.xacro (robot description, xacro)
@@ -86,5 +86,5 @@
     <parent link="world"/>
     <child link="cube"/>
-    <origin xyz="0.0 0.65 0.2" rpy="0 0 3.1415"/>
+    <origin xyz="0.0 0.65 0.0" rpy="0 0 3.1415"/>
     </joint>
   <gazebo reference="world">
